File: hardware/irouette.kicad_pcb (KiCad board)
At the start: 2 copper layers, 80 x 35.6 mm, 20 parts, among them J1 Screw_Terminal_01x02, J2 Screw_Terminal_01x02, J3 Screw_Terminal_01x02, Q1 PMOS_SI2302, U1 ESP32-WROOM, U2 TP4056, U3 HT7333

Commit message: Updated libs
Parts:
- added C6: 100n, Capacitor_SMD:C_0805_2012Metric_Pad1.15x1.40mm_HandSolder, F.Cu at (66.6, 45.3)
- added Q2: SI2301, Package_TO_SOT_SMD:SOT-23, F.Cu at (71.3, 44.4)
- added R5: 100, Resistor_SMD:R_0805_2012Metric_Pad1.15x1.40mm_HandSolder, F.Cu at (71.5, 41.6)
- added U4: DW01, Package_TO_SOT_SMD:SOT-23-6_Handsoldering, F.Cu at (67.2, 42.5)
- D1: value 1N5818 -> TL431LP; footprint Diode_SMD:D_SMA_Handsoldering -> Package_TO_SOT_THT:TO-92_Inline
- D3: value TL431LP -> 1N5818; footprint Package_TO_SOT_THT:TO-92_Inline -> Diode_SMD:D_SMA_Handsoldering
- Q1: footprint Package_TO_SOT_SMD:SOT-23-5_HandSoldering -> Package_TO_SOT_SMD:SOT-23
- R3: value R_US -> 1.2k
- R4: value R_US -> 1k
- U1: value ESP32-WROOM -> HT7333; footprint ESP32-footprints-Lib:ESP32-WROOM -> Package_TO_SOT_SMD:SOT-89-3_Handsoldering
- U3: value HT7333 -> FS8205A; footprint Package_TO_SOT_SMD:SOT-89-3_Handsoldering -> Package_SO:TSSOP-8_4.4x3mm_P0.65mm
Connections:
- C2 pad 1: Net-(C2-Pad1) -> (no net)
- C5 pad 1: +3V3 -> Net-(C5-Pad1)
- C5 pad 2: GND -> /VBAT_GND
- D1 pad 1: /Vpanel -> (no net)
- D1 pad 2: Net-(D1-Pad2) -> (no net)
- D3 pad 1: Net-(D3-Pad1) -> /Vpanel
- J1 pad 2: Net-(D1-Pad2) -> Net-(D2-Pad2)
- J2 pad 2: Net-(D2-Pad2) -> Net-(D3-Pad2)
- J3 pad 2: GND -> /VBAT_GND
- Q1 pad 1: Net-(Q1-Pad1) -> (no net)
- Q1 pad 2: Net-(Q1-Pad2) -> (no net)
- Q1 pad 3: Net-(Q1-Pad3) -> (no net)
- R4 pad 1: Net-(R3-Pad1) -> Net-(R4-Pad1)
- R4 pad 2: Net-(R3-Pad2) -> GND
- U1 pad 2: +3V3 -> Net-(JP1-Pad2)
- U2 pad 6: Net-(U2-Pad6) -> (no net)
- U2 pad 7: Net-(U2-Pad7) -> (no net)
- U3 pad 1: GND -> (no net)
- U3 pad 2: Net-(JP1-Pad2) -> /VBAT_GND
- U3 pad 3: +3V3 -> /VBAT_GND

Commit message: up
Parts:
- added U5: ESP32-WROOM, custom:esp32_wroom, F.Cu at (86.1, 60.9)
- moved U1 16.6 mm to (94.0, 41.9)
Changed lines of the file:
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@@
     (tracks 0)
     (zones 0)
-    (modules 24)
+    (modules 25)
     (nets 15)
   )
@@
   )
   (module Package_TO_SOT_SMD:SOT-89-3_Handsoldering (layer F.Cu)
-    (at 84.79 55.79)
+    (at 93.98 41.91)
     (descr "SOT-89-3 Handsoldering")
     (tags "SOT-89-3 Handsoldering")
@@
     )
   )
+  (module custom:esp32_wroom (layer F.Cu)
+    (at 86.06 60.87)
+    (fp_text reference U5 (at -11.557 9.017) (layer F.SilkS)
+      (effects (font (size 1 1) (thickness 0.15)))
+    )
+    (fp_text value ESP32-WROOM (at 5.715 14.224) (layer F.Fab)
+      (effects (font (size 1 1) (thickness 0.15)))
+    )
+    (fp_text user "Espressif Systems" (at -6.858 -0.889 90) (layer F.SilkS)
+      (effects (font (size 1 1) (thickness 0.15)))
+    )
+    (fp_circle (center 9.906 6.604) (end 10.033 6.858) (layer F.SilkS) (width 0.5))
+    (fp_text user ESP32-WROOM (at -5.207 0.254 90) (layer F.SilkS)
+      (effects (font (size 1 1) (thickness 0.15)))
+    )
+    (fp_line (start -9 6.75) (end 9 6.75) (layer F.SilkS) (width 0.15))
+    (fp_line (start 9 12.75) (end 9 -12.75) (layer F.SilkS) (width 0.15))
+    (fp_line (start -9 12.75) (end -9 -12.75) (layer F.SilkS) (width 0.15))
+    (fp_line (start -9 -12.75) (end 9 -12.75) (layer F.SilkS) (width 0.15))
+    (fp_line (start -9 12.75) (end 9 12.75) (layer F.SilkS) (width 0.15))
+    (pad 38 smd oval (at -9 5.25) (size 2.5 0.9) (layers F.Cu F.Paste F.Mask)
+      (net 4 GND))
+    (pad 37 smd oval (at -9 3.98) (size 2.5 0.9) (layers F.Cu F.Paste F.Mask))
+    (pad 36 smd oval (at -9 2.71) (size 2.5 0.9) (layers F.Cu F.Paste F.Mask))
+    (pad 35 smd oval (at -9 1.44) (size 2.5 0.9) (layers F.Cu F.Paste F.Mask))
+    (pad 34 smd oval (at -9 0.17) (size 2.5 0.9) (layers F.Cu F.Paste F.Mask))
+    (pad 33 smd oval (at -9 -1.1) (size 2.5 0.9) (layers F.Cu F.Paste F.Mask))
+    (pad 32 smd oval (at -9 -2.37) (size 2.5 0.9) (layers F.Cu F.Paste F.Mask))
+    (pad 31 smd oval (at -9 -3.64) (size 2.5 0.9) (layers F.Cu F.Paste F.Mask))
+    (pad 30 smd oval (at -9 -4.91) (size 2.5 0.9) (layers F.Cu F.Paste F.Mask))
+    (pad 29 smd oval (at -9 -6.18) (size 2.5 0.9) (layers F.Cu F.Paste F.Mask))
+    (pad 28 smd oval (at -9 -7.45) (size 2.5 0.9) (layers F.Cu F.Paste F.Mask))
+    (pad 27 smd oval (at -9 -8.72) (size 2.5 0.9) (layers F.Cu F.Paste F.Mask))
+    (pad 26 smd oval (at -9 -9.99) (size 2.5 0.9) (layers F.Cu F.Paste F.Mask))
+    (pad 25 smd oval (at -9 -11.26) (size 2.5 0.9) (layers F.Cu F.Paste F.Mask))
+    (pad 24 smd oval (at -5.715 -12.75) (size 0.9 2.5) (layers F.Cu F.Paste F.Mask))
+    (pad 23 smd oval (at -4.445 -12.75) (size 0.9 2.5) (layers F.Cu F.Paste F.Mask))
+    (pad 22 smd oval (at -3.175 -12.75) (size 0.9 2.5) (layers F.Cu F.Paste F.Mask))
+    (pad 21 smd oval (at -1.905 -12.75) (size 0.9 2.5) (layers F.Cu F.Paste F.Mask))
+    (pad 20 smd oval (at -0.635 -12.75) (size 0.9 2.5) (layers F.Cu F.Paste F.Mask))
+    (pad 19 smd oval (at 0.635 -12.75) (size 0.9 2.5) (layers F.Cu F.Paste F.Mask))
+    (pad 18 smd oval (at 1.905 -12.75) (size 0.9 2.5) (layers F.Cu F.Paste F.Mask))
+    (pad 17 smd oval (at 3.175 -12.75) (size 0.9 2.5) (layers F.Cu F.Paste F.Mask))
+    (pad 16 smd oval (at 4.445 -12.75) (size 0.9 2.5) (layers F.Cu F.Paste F.Mask))
+    (pad 15 smd oval (at 5.715 -12.75) (size 0.9 2.5) (layers F.Cu F.Paste F.Mask)
+      (net 4 GND))
+    (pad 14 smd oval (at 9 -11.26) (size 2.5 0.9) (layers F.Cu F.Paste F.Mask))
+    (pad 13 smd oval (at 9 -9.99) (size 2.5 0.9) (layers F.Cu F.Paste F.Mask))
+    (pad 12 smd oval (at 9 -8.72) (size 2.5 0.9) (layers F.Cu F.Paste F.Mask))
+    (pad 11 smd oval (at 9 -7.45) (size 2.5 0.9) (layers F.Cu F.Paste F.Mask))
+    (pad 10 smd oval (at 9 -6.18) (size 2.5 0.9) (layers F.Cu F.Paste F.Mask))
+    (pad 9 smd oval (at 9 -4.91) (size 2.5 0.9) (layers F.Cu F.Paste F.Mask))
+    (pad 8 smd oval (at 9 -3.64) (size 2.5 0.9) (layers F.Cu F.Paste F.Mask))
+    (pad 7 smd oval (at 9 -2.37) (size 2.5 0.9) (layers F.Cu F.Paste F.Mask))
+    (pad 6 smd oval (at 9 -1.1) (size 2.5 0.9) (layers F.Cu F.Paste F.Mask))
+    (pad 5 smd oval (at 9 0.17) (size 2.5 0.9) (layers F.Cu F.Paste F.Mask))
+    (pad 4 smd oval (at 9 1.44) (size 2.5 0.9) (layers F.Cu F.Paste F.Mask))
+    (pad 3 smd oval (at 9 2.71) (size 2.5 0.9) (layers F.Cu F.Paste F.Mask)
+      (net 7 +3V3))
+    (pad 2 smd oval (at 9 3.98) (size 2.5 0.9) (layers F.Cu F.Paste F.Mask)
+      (net 7 +3V3))
+    (pad 1 smd oval (at 9 5.25) (size 2.5 0.9) (layers F.Cu F.Paste F.Mask)
+      (net 4 GND))
+    (pad 39 smd rect (at 0.3 -2.45) (size 6 6) (layers F.Cu F.Paste F.Mask)
+      (net 4 GND))
+  )
   (gr_line (start 25.4 73.66) (end 25.4 38.1) (layer Edge.Cuts) (width 0.15))
