File: hardware/irouette.kicad_pcb (KiCad board)
At the start: 2 copper layers, 80 x 35.6 mm, 25 parts, among them J1 Screw_Terminal_01x02, J2 Screw_Terminal_01x02, J3 Screw_Terminal_01x02, Q1 PMOS_SI2302, Q2 SI2301, U1 HT7333, U2 TP4056, U3 FS8205A, U4 DW01, U5 ESP32-WROOM

Commit message: Update schematic with vcc peripheral generation
Parts:
- added D4: LED_VCC33_PER, LEDs:LED_0805_HandSoldering, F.Cu at (55.9, 62.2)
Connections:
- C2 pad 1: (no net) -> Net-(C2-Pad1)
- D1 pad 1: (no net) -> /VREF_2.5
- D1 pad 2: (no net) -> GND
- D1 pad 3: (no net) -> /VREF_2.5
- Q1 pad 1: (no net) -> Net-(Q1-Pad1)
- Q1 pad 2: (no net) -> Net-(Q1-Pad2)
- Q1 pad 3: (no net) -> Net-(Q1-Pad3)
- Q2 pad 1: (no net) -> /VCC33_PER_CMD
- Q2 pad 2: (no net) -> +3V3
- Q2 pad 3: (no net) -> /VCC33_PER
- U2 pad 6: (no net) -> Net-(U2-Pad6)
- U2 pad 7: (no net) -> Net-(U2-Pad7)
- U3 pad 1: (no net) -> Net-(U3-Pad1)
- U3 pad 8: (no net) -> Net-(U3-Pad8)
- U4 pad 4: (no net) -> Net-(U4-Pad4)
- U5 pad 10: (no net) -> Net-(U5-Pad10)
- U5 pad 11: (no net) -> Net-(U5-Pad11)
- U5 pad 12: (no net) -> Net-(U5-Pad12)
- U5 pad 13: (no net) -> Net-(U5-Pad13)
- U5 pad 14: (no net) -> Net-(U5-Pad14)
- U5 pad 16: (no net) -> Net-(U5-Pad16)
- U5 pad 17: (no net) -> Net-(U5-Pad17)
- U5 pad 18: (no net) -> Net-(U5-Pad18)
- U5 pad 19: (no net) -> Net-(U5-Pad19)
- U5 pad 20: (no net) -> Net-(U5-Pad20)
- U5 pad 21: (no net) -> Net-(U5-Pad21)
- U5 pad 22: (no net) -> Net-(U5-Pad22)
- U5 pad 23: (no net) -> Net-(U5-Pad23)
- U5 pad 24: (no net) -> Net-(U5-Pad24)
- U5 pad 25: (no net) -> Net-(U5-Pad25)
- U5 pad 26: (no net) -> Net-(U5-Pad26)
- U5 pad 27: (no net) -> Net-(U5-Pad27)
- U5 pad 28: (no net) -> Net-(U5-Pad28)
- U5 pad 29: (no net) -> Net-(U5-Pad29)
- U5 pad 30: (no net) -> Net-(U5-Pad30)
- U5 pad 31: (no net) -> Net-(U5-Pad31)
- U5 pad 32: (no net) -> Net-(U5-Pad32)
- U5 pad 33: (no net) -> Net-(U5-Pad33)
- U5 pad 34: (no net) -> Net-(U5-Pad34)
- U5 pad 35: (no net) -> Net-(U5-Pad35)
- U5 pad 36: (no net) -> Net-(U5-Pad36)
- U5 pad 37: (no net) -> Net-(U5-Pad37)
- U5 pad 4: (no net) -> Net-(U5-Pad4)
- U5 pad 5: (no net) -> Net-(U5-Pad5)
- U5 pad 6: (no net) -> Net-(U5-Pad6)
- U5 pad 7: (no net) -> Net-(U5-Pad7)
- U5 pad 8: (no net) -> Net-(U5-Pad8)
- U5 pad 9: (no net) -> Net-(U5-Pad9)

Commit message: Changed LED
Parts:
- added R6: 100k, Resistor_SMD:R_0805_2012Metric_Pad1.15x1.40mm_HandSolder, F.Cu at (66.6, 61.9)
- added R7: 1k, Resistor_SMD:R_0805_2012Metric_Pad1.15x1.40mm_HandSolder, F.Cu at (66.6, 63.9)
- added R8: 100k, Resistor_SMD:R_0805_2012Metric_Pad1.15x1.40mm_HandSolder, F.Cu at (70.4, 61.9)
- D1: footprint Package_TO_SOT_THT:TO-92_Inline -> Package_TO_SOT_SMD:SOT-23
- D4: footprint LEDs:LED_0805_HandSoldering -> LED_SMD:LED_0805_2012Metric
Connections:
- C2 pad 1: Net-(C2-Pad1) -> (no net)
- Q1 pad 1: Net-(Q1-Pad1) -> (no net)
- Q1 pad 2: Net-(Q1-Pad2) -> (no net)
- Q1 pad 3: Net-(Q1-Pad3) -> (no net)
- U2 pad 6: Net-(U2-Pad6) -> (no net)
- U2 pad 7: Net-(U2-Pad7) -> (no net)
- U3 pad 1: Net-(U3-Pad1) -> (no net)
- U3 pad 8: Net-(U3-Pad8) -> (no net)
- U4 pad 4: Net-(U4-Pad4) -> (no net)
- U5 pad 10: Net-(U5-Pad10) -> (no net)
- U5 pad 11: Net-(U5-Pad11) -> (no net)
- U5 pad 12: Net-(U5-Pad12) -> (no net)
- U5 pad 13: Net-(U5-Pad13) -> (no net)
- U5 pad 14: Net-(U5-Pad14) -> (no net)
- U5 pad 16: Net-(U5-Pad16) -> (no net)
- U5 pad 17: Net-(U5-Pad17) -> (no net)
- U5 pad 18: Net-(U5-Pad18) -> (no net)
- U5 pad 19: Net-(U5-Pad19) -> (no net)
- U5 pad 20: Net-(U5-Pad20) -> (no net)
- U5 pad 21: Net-(U5-Pad21) -> (no net)
- U5 pad 22: Net-(U5-Pad22) -> (no net)
- U5 pad 23: Net-(U5-Pad23) -> (no net)
- U5 pad 24: Net-(U5-Pad24) -> (no net)
- U5 pad 25: Net-(U5-Pad25) -> (no net)
- U5 pad 26: Net-(U5-Pad26) -> (no net)
- U5 pad 27: Net-(U5-Pad27) -> (no net)
- U5 pad 28: Net-(U5-Pad28) -> (no net)
- U5 pad 29: Net-(U5-Pad29) -> (no net)
- U5 pad 30: Net-(U5-Pad30) -> (no net)
- U5 pad 31: Net-(U5-Pad31) -> (no net)
- U5 pad 32: Net-(U5-Pad32) -> (no net)
- U5 pad 33: Net-(U5-Pad33) -> (no net)
- U5 pad 34: Net-(U5-Pad34) -> (no net)
- U5 pad 35: Net-(U5-Pad35) -> (no net)
- U5 pad 36: Net-(U5-Pad36) -> (no net)
- U5 pad 37: Net-(U5-Pad37) -> (no net)
- U5 pad 4: Net-(U5-Pad4) -> (no net)
- U5 pad 5: Net-(U5-Pad5) -> (no net)
- U5 pad 6: Net-(U5-Pad6) -> (no net)
- U5 pad 7: Net-(U5-Pad7) -> (no net)
- U5 pad 8: Net-(U5-Pad8) -> (no net)
- U5 pad 9: Net-(U5-Pad9) -> (no net)

Commit message: Adding sensoes
Parts:
- added R10: 100k, Resistor_SMD:R_0805_2012Metric_Pad1.15x1.40mm_HandSolder, F.Cu at (56.5, 70.2)
- added R9: 100k, Resistor_SMD:R_0805_2012Metric_Pad1.15x1.40mm_HandSolder, F.Cu at (56.5, 68.3)
- added U7: BMP180, custom:BMP180, F.Cu at (61.0, 71.1)
Changed lines of the file:
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@@
     (tracks 0)
     (zones 0)
-    (modules 29)
-    (nets 19)
+    (modules 32)
+    (nets 21)
   )
   (page A4)
@@
   (net 17 /VCC33_PER_CMD)
   (net 18 /VCC33_PER)
+  (net 19 /SDA)
+  (net 20 /SCL)
   (net_class Default "Ceci est la Netclass par défaut."
     (clearance 0.2)
@@
     (uvia_drill 0.1)
     (add_net +3V3)
+    (add_net /SCL)
+    (add_net /SDA)
     (add_net /VBAT)
     (add_net /VBAT_DIV2)
@@
     )
   )
+  (module Resistor_SMD:R_0805_2012Metric_Pad1.15x1.40mm_HandSolder (layer F.Cu)
+    (at 56.485001 68.285001)
+    (descr "Resistor SMD 0805 (2012 Metric), square (rectangular) end terminal, IPC_7351 nominal with elongated pad for handsoldering. (Body size source: https://docs.google.com/spreadsheets/d/1BsfQQcO9C6DZCsRaXUlFlo91Tg2WpOkGARC1WS5S8t0/edit?usp=sharing), generated with kicad-footprint-generator")
+    (tags "resistor handsolder")
+    (attr smd)
+    (fp_text reference R9 (at 0 -1.65) (layer F.SilkS)
+      (effects (font (size 1 1) (thickness 0.15)))
+    )
+    (fp_text value 100k (at 0 1.65) (layer F.Fab)
+      (effects (font (size 1 1) (thickness 0.15)))
+    )
+    (fp_text user %R (at 0 0) (layer F.Fab)
+      (effects (font (size 0.5 0.5) (thickness 0.08)))
+    )
+    (fp_line (start 1.85 0.95) (end -1.85 0.95) (layer F.CrtYd) (width 0.05))
+    (fp_line (start 1.85 -0.95) (end 1.85 0.95) (layer F.CrtYd) (width 0.05))
+    (fp_line (start -1.85 -0.95) (end 1.85 -0.95) (layer F.CrtYd) (width 0.05))
+    (fp_line (start -1.85 0.95) (end -1.85 -0.95) (layer F.CrtYd) (width 0.05))
+    (fp_line (start -0.261252 0.71) (end 0.261252 0.71) (layer F.SilkS) (width 0.12))
+    (fp_line (start -0.261252 -0.71) (end 0.261252 -0.71) (layer F.SilkS) (width 0.12))
+    (fp_line (start 1 0.6) (end -1 0.6) (layer F.Fab) (width 0.1))
+    (fp_line (start 1 -0.6) (end 1 0.6) (layer F.Fab) (width 0.1))
+    (fp_line (start -1 -0.6) (end 1 -0.6) (layer F.Fab) (width 0.1))
+    (fp_line (start -1 0.6) (end -1 -0.6) (layer F.Fab) (width 0.1))
+    (pad 2 smd roundrect (at 1.025 0) (size 1.15 1.4) (layers F.Cu F.Paste F.Mask) (roundrect_rratio 0.217391)
+      (net 19 /SDA))
+    (pad 1 smd roundrect (at -1.025 0) (size 1.15 1.4) (layers F.Cu F.Paste F.Mask) (roundrect_rratio 0.217391)
+      (net 18 /VCC33_PER))
+    (model ${KISYS3DMOD}/Resistor_SMD.3dshapes/R_0805_2012Metric.wrl
+      (at (xyz 0 0 0))
+      (scale (xyz 1 1 1))
+      (rotate (xyz 0 0 0))
+    )
+  )
+  (module Resistor_SMD:R_0805_2012Metric_Pad1.15x1.40mm_HandSolder (layer F.Cu)
+    (at 56.485001 70.235001)
+    (descr "Resistor SMD 0805 (2012 Metric), square (rectangular) end terminal, IPC_7351 nominal with elongated pad for handsoldering. (Body size source: https://docs.google.com/spreadsheets/d/1BsfQQcO9C6DZCsRaXUlFlo91Tg2WpOkGARC1WS5S8t0/edit?usp=sharing), generated with kicad-footprint-generator")
+    (tags "resistor handsolder")
+    (attr smd)
+    (fp_text reference R10 (at 0 -1.65) (layer F.SilkS)
+      (effects (font (size 1 1) (thickness 0.15)))
+    )
+    (fp_text value 100k (at 0 1.65) (layer F.Fab)
+      (effects (font (size 1 1) (thickness 0.15)))
+    )
+    (fp_line (start -1 0.6) (end -1 -0.6) (layer F.Fab) (width 0.1))
+    (fp_line (start -1 -0.6) (end 1 -0.6) (layer F.Fab) (width 0.1))
+    (fp_line (start 1 -0.6) (end 1 0.6) (layer F.Fab) (width 0.1))
+    (fp_line (start 1 0.6) (end -1 0.6) (layer F.Fab) (width 0.1))
+    (fp_line (start -0.261252 -0.71) (end 0.261252 -0.71) (layer F.SilkS) (width 0.12))
+    (fp_line (start -0.261252 0.71) (end 0.261252 0.71) (layer F.SilkS) (width 0.12))
+    (fp_line (start -1.85 0.95) (end -1.85 -0.95) (layer F.CrtYd) (width 0.05))
+    (fp_line (start -1.85 -0.95) (end 1.85 -0.95) (layer F.CrtYd) (width 0.05))
+    (fp_line (start 1.85 -0.95) (end 1.85 0.95) (layer F.CrtYd) (width 0.05))
+    (fp_line (start 1.85 0.95) (end -1.85 0.95) (layer F.CrtYd) (width 0.05))
+    (fp_text user %R (at 0 0) (layer F.Fab)
+      (effects (font (size 0.5 0.5) (thickness 0.08)))
+    )
+    (pad 1 smd roundrect (at -1.025 0) (size 1.15 1.4) (layers F.Cu F.Paste F.Mask) (roundrect_rratio 0.217391)
+      (net 18 /VCC33_PER))
+    (pad 2 smd roundrect (at 1.025 0) (size 1.15 1.4) (layers F.Cu F.Paste F.Mask) (roundrect_rratio 0.217391)
+      (net 20 /SCL))
+    (model ${KISYS3DMOD}/Resistor_SMD.3dshapes/R_0805_2012Metric.wrl
+      (at (xyz 0 0 0))
+      (scale (xyz 1 1 1))
+      (rotate (xyz 0 0 0))
+    )
+  )
+  (module custom:BMP180 (layer F.Cu)
+    (at 60.96 71.12)
+    (fp_text reference U7 (at 1.27 2.54) (layer F.SilkS)
+      (effects (font (size 1 1) (thickness 0.15)))
+    )
+    (fp_text value BMP180 (at 2.54 -2.54) (layer F.Fab)
+      (effects (font (size 1 1) (thickness 0.15)))
+    )
+    (fp_line (start -1.27 1.27) (end 12.7 1.27) (layer F.SilkS) (width 0.15))
+    (fp_line (start 12.7 1.27) (end 12.7 -7.62) (layer F.SilkS) (width 0.15))
+    (fp_line (start 12.7 -7.62) (end -2.54 -7.62) (layer F.SilkS) (width 0.15))
+    (fp_line (start -2.54 -7.62) (end -2.54 1.27) (layer F.SilkS) (width 0.15))
+    (fp_line (start -2.54 1.27) (end -1.27 1.27) (layer F.SilkS) (width 0.15))
+    (fp_line (start -2.54 2.54) (end -2.54 -8.89) (layer F.CrtYd) (width 0.15))
+    (fp_line (start -2.54 -8.89) (end 12.7 -8.89) (layer F.CrtYd) (width 0.15))
+    (fp_line (start 12.7 -8.89) (end 12.7 2.54) (layer F.CrtYd) (width 0.15))
+    (fp_line (start 12.7 2.54) (end -2.54 2.54) (layer F.CrtYd) (width 0.15))
+    (pad 1 thru_hole circle (at 0 0) (size 1.524 1.524) (drill 0.762) (layers *.Cu *.Mask)
+      (net 18 /VCC33_PER))
+    (pad 2 thru_hole circle (at 2.54 0) (size 1.524 1.524) (drill 0.762) (layers *.Cu *.Mask)
+      (net 4 GND))
+    (pad 3 thru_hole circle (at 5.08 0) (size 1.524 1.524) (drill 0.762) (layers *.Cu *.Mask)
+      (net 20 /SCL))
+    (pad 4 thru_hole circle (at 7.62 0) (size 1.524 1.524) (drill 0.762) (layers *.Cu *.Mask)
+      (net 19 /SDA))
+    (pad 5 thru_hole circle (at 10.16 0) (size 1.524 1.524) (drill 0.762) (layers *.Cu *.Mask))
+  )
   (gr_line (start 25.4 73.66) (end 25.4 38.1) (layer Edge.Cuts) (width 0.15))
