File: hardware/irouette.sch (KiCad schematic (older format))
At the start: 20 parts, among them J1 Screw_Terminal_01x02, J2 Screw_Terminal_01x02, J3 Screw_Terminal_01x02, Q1 PMOS_SI2302, Q2 SI2301, U1 ESP32-WROOM, U2 TP4056, U3 HT7333

Commit message: Updated libs
Parts:
- added C5: 100n, Capacitor_SMD:C_0805_2012Metric_Pad1.15x1.40mm_HandSolder, symbol Device:C
- added R4: 1k, Resistor_SMD:R_0805_2012Metric_Pad1.15x1.40mm_HandSolder, symbol Device:R_US
- added R5: 100, Resistor_SMD:R_0805_2012Metric_Pad1.15x1.40mm_HandSolder, symbol Device:R_US
- added U3: FS8205A, Package_SO:TSSOP-8_4.4x3mm_P0.65mm, symbol custom_lib:FS8205A
- added U4: DW01, Package_TO_SOT_SMD:SOT-23-6_Handsoldering, symbol custom_lib:DW01
- Q1: footprint Package_TO_SOT_SMD:SOT-23-5_HandSoldering -> Package_TO_SOT_SMD:SOT-23
- Q2: footprint (none) -> Package_TO_SOT_SMD:SOT-23
- R3: value R_US -> 1.2k
- renumbered C5 to C6, D3 to D1, D1 to D2, D2 to D3, U3 to U1, U1 to U5
Connections:
- net GND: now also R4.2, U3.6 (S2), U3.7 (S2); no longer J3.2 (Pin_2)
- net VBAT: now also R5.1
- new net: U3.4 (G1), U4.1 (OD)
- new net: R4.1, U4.2 (CS)
- new net: U3.5 (G2), U4.3 (OC)
- new net: C5.1, R5.2, U4.5 (VCC)
- new net VBAT_GND: C5.2, J3.2 (Pin_2), U3.2 (S1), U3.3 (S1), U4.6 (GND)
- no-connect marks 2 -> 5
Other:
- moved on the sheet: J3
Changed lines of the file:
@@
 $EndDescr
 $Comp
-L custom_lib:ESP-32U U1
+L custom_lib:ESP-32U U5
 U 1 1 5BF317FE
 P 6450 4550
-F 0 "U1" H 6425 5937 60  0000 C CNN
+F 0 "U5" H 6425 5937 60  0000 C CNN
 F 1 "ESP32-WROOM" H 6425 5831 60  0000 C CNN
 F 2 "ESP32-footprints-Lib:ESP32-WROOM" H 6800 5900 60  0001 C CNN
@@
 $EndComp
 $Comp
-L Diode:1N5818 D1
+L Diode:1N5818 D2
 U 1 1 5BFC508E
 P 1500 850
-F 0 "D1" H 1500 726 50  0000 C CNN
+F 0 "D2" H 1500 726 50  0000 C CNN
 F 1 "1N5818" H 1500 725 50  0001 C CNN
 F 2 "Diode_SMD:D_SMA_Handsoldering" H 1500 675 50  0001 C CNN
@@
 $EndComp
 $Comp
-L Diode:1N5818 D2
+L Diode:1N5818 D3
 U 1 1 5BFC532C
 P 1500 1200
-F 0 "D2" H 1500 1076 50  0000 C CNN
+F 0 "D3" H 1500 1076 50  0000 C CNN
 F 1 "1N5818" H 1500 1075 50  0001 C CNN
 F 2 "Diode_SMD:D_SMA_Handsoldering" H 1500 1025 50  0001 C CNN
@@
 L Connector:Screw_Terminal_01x02 J3
 U 1 1 5BFC56EB
-P 3600 850
-F 0 "J3" H 3650 650 50  0000 C CNN
-F 1 "Screw_Terminal_01x02" H 3650 950 50  0001 C CNN
-F 2 "TerminalBlock:TerminalBlock_bornier-2_P5.08mm" H 3600 850 50  0001 C CNN
-F 3 "~" H 3600 850 50  0001 C CNN
-	1    3600 850
+P 6000 850
+F 0 "J3" H 6050 650 50  0000 C CNN
+F 1 "Screw_Terminal_01x02" H 6050 950 50  0001 C CNN
+F 2 "TerminalBlock:TerminalBlock_bornier-2_P5.08mm" H 6000 850 50  0001 C CNN
+F 3 "~" H 6000 850 50  0001 C CNN
+	1    6000 850
 	1    0    0    -1
 $EndComp
@@
 Wire Wire Line
 	2700 1500 2800 1500
-Wire Wire Line
-	3150 850  3400 850
 Text Label 3150 850  0    50   ~ 0
 VBAT
@@
 Wire Wire Line
 	3150 950  3150 1150
-Connection ~ 3400 950
 $Comp
 L power:GND #PWR011
@@
 P 3150 1400
 F 0 "R3" H 3218 1446 50  0000 L CNN
-F 1 "R_US" H 3218 1355 50  0000 L CNN
+F 1 "1.2k" H 3218 1355 50  0000 L CNN
 F 2 "Resistor_SMD:R_0805_2012Metric_Pad1.15x1.40mm_HandSolder" V 3190 1390 50  0001 C CNN
 F 3 "~" H 3150 1400 50  0001 C CNN
@@
 VBAT_DIV2
 $Comp
-L custom_lib:HT7333 U3
+L custom_lib:HT7333 U1
 U 1 1 5BFC9A88
 P 1850 2650
-F 0 "U3" H 2125 3215 50  0000 C CNN
+F 0 "U1" H 2125 3215 50  0000 C CNN
 F 1 "HT7333" H 2125 3124 50  0000 C CNN
 F 2 "Package_TO_SOT_SMD:SOT-89-3_Handsoldering" H 1850 2650 50  0001 C CNN
@@
 $EndComp
 $Comp
-L power:+3.3V #PWR013
+L power:+3.3V #PWR015
 U 1 1 5BFCB093
 P 4800 3900
-F 0 "#PWR013" H 4800 3750 50  0001 C CNN
+F 0 "#PWR015" H 4800 3750 50  0001 C CNN
 F 1 "+3.3V" H 4815 4073 50  0000 C CNN
 F 2 "" H 4800 3900 50  0001 C CNN
@@
 	5200 3950 4800 3950
 $Comp
-L power:GND #PWR014
+L power:GND #PWR018
 U 1 1 5BFCBAF4
 P 5400 3800
-F 0 "#PWR014" H 5400 3550 50  0001 C CNN
+F 0 "#PWR018" H 5400 3550 50  0001 C CNN
 F 1 "GND" H 5250 3750 50  0000 C CNN
 F 2 "" H 5400 3800 50  0001 C CNN
@@
 	5500 3800 5500 3850
 $Comp
-L power:GND #PWR016
+L power:GND #PWR020
 U 1 1 5BFCC293
 P 7600 3800
-F 0 "#PWR016" H 7600 3550 50  0001 C CNN
+F 0 "#PWR020" H 7600 3550 50  0001 C CNN
 F 1 "GND" H 7750 3750 50  0000 C CNN
 F 2 "" H 7600 3800 50  0001 C CNN
@@
 	7450 3800 7350 3800
 $Comp
-L power:GND #PWR015
+L power:GND #PWR019
 U 1 1 5BFCCB77
 P 6000 5650
-F 0 "#PWR015" H 6000 5400 50  0001 C CNN
+F 0 "#PWR019" H 6000 5400 50  0001 C CNN
 F 1 "GND" H 5850 5600 50  0000 C CNN
 F 2 "" H 6000 5650 50  0001 C CNN
@@
 NoConn ~ 2700 2600
 $Comp
-L Device:C C5
+L Device:C C6
 U 1 1 5BFCE1AC
 P 5200 3400
-F 0 "C5" H 5315 3446 50  0000 L CNN
+F 0 "C6" H 5315 3446 50  0000 L CNN
 F 1 "100n" H 5315 3355 50  0000 L CNN
 F 2 "Capacitor_SMD:C_0805_2012Metric_Pad1.15x1.40mm_HandSolder" H 5238 3250 50  0001 C CNN
@@
 $EndComp
 $Comp
-L power:+3.3V #PWR0101
+L power:+3.3V #PWR016
 U 1 1 5BFCE2B3
 P 5200 3250
-F 0 "#PWR0101" H 5200 3100 50  0001 C CNN
+F 0 "#PWR016" H 5200 3100 50  0001 C CNN
 F 1 "+3.3V" H 5215 3423 50  0000 C CNN
 F 2 "" H 5200 3250 50  0001 C CNN
@@
 $EndComp
 $Comp
-L power:GND #PWR0102
+L power:GND #PWR017
 U 1 1 5BFCE2E0
 P 5200 3550
-F 0 "#PWR0102" H 5200 3300 50  0001 C CNN
+F 0 "#PWR017" H 5200 3300 50  0001 C CNN
 F 1 "GND" H 5050 3500 50  0000 C CNN
 F 2 "" H 5200 3550 50  0001 C CNN
@@
 $EndComp
 $Comp
-L Reference_Voltage:TL431LP D3
+L Reference_Voltage:TL431LP D1
 U 1 1 5BFCF494
 P 1350 4750
-F 0 "D3" V 1396 4681 50  0000 R CNN
+F 0 "D1" V 1396 4681 50  0000 R CNN
 F 1 "TL431LP" V 1305 4681 50  0000 R CNN
 F 2 "Package_TO_SOT_THT:TO-92_Inline" H 1350 4600 50  0001 C CIN
@@
 F 0 "Q2" H 4105 3146 50  0000 L CNN
 F 1 "SI2301" H 4105 3055 50  0000 L CNN
-F 2 "" H 4100 3200 50  0001 C CNN
+F 2 "Package_TO_SOT_SMD:SOT-23" H 4100 3200 50  0001 C CNN
 F 3 "~" H 3900 3100 50  0001 C CNN
 	1    3900 3100
@@
 F 0 "Q1" V 3143 3500 50  0000 C CNN
 F 1 "PMOS_SI2302" V 3052 3500 50  0000 C CNN
-F 2 "Package_TO_SOT_SMD:SOT-23-5_HandSoldering" H 3000 3600 50  0001 C CNN
+F 2 "Package_TO_SOT_SMD:SOT-23" H 3000 3600 50  0001 C CNN
 F 3 "~" H 2800 3500 50  0001 C CNN
 	1    2800 3500
 	0    1    -1   0
 $EndComp
+$Comp
+L custom_lib:DW01 U4
+U 1 1 5C0989E7
+P 3950 1550
+F 0 "U4" H 4000 1600 50  0000 C CNN
+F 1 "DW01" H 4300 1700 50  0000 C CNN
+F 2 "Package_TO_SOT_SMD:SOT-23-6_Handsoldering" H 3800 1400 50  0001 C CNN
+F 3 "" H 3800 1400 50  0001 C CNN
+	1    3950 1550
+	1    0    0    -1
+$EndComp
+$Comp
+L custom_lib:FS8205A U3
+U 1 1 5C098A78
+P 3750 2500
+F 0 "U3" H 3800 2450 50  0000 C CNN
+F 1 "FS8205A" H 4600 2450 50  0000 C CNN
+F 2 "Package_SO:TSSOP-8_4.4x3mm_P0.65mm" H 3750 2500 50  0001 C CNN
+F 3 "" H 3750 2500 50  0001 C CNN
+	1    3750 2500
+	1    0    0    -1
+$EndComp
+$Comp
+L Device:R_US R4
+U 1 1 5C099C2F
+P 3700 1350
+F 0 "R4" H 3768 1396 50  0000 L CNN
+F 1 "1k" H 3768 1305 50  0000 L CNN
+F 2 "Resistor_SMD:R_0805_2012Metric_Pad1.15x1.40mm_HandSolder" V 3740 1340 50  0001 C CNN
+F 3 "~" H 3700 1350 50  0001 C CNN
+	1    3700 1350
+	1    0    0    -1
+$EndComp
+Wire Wire Line
+	4500 1550 4500 1700
+Wire Wire Line
+	4500 1700 4550 1700
+Wire Wire Line
+	4550 1700 4550 1800
+Wire Wire Line
+	4150 1550 4150 1700
+Wire Wire Line
+	4150 1700 4050 1700
+Wire Wire Line
+	4050 1700 4050 1800
+NoConn ~ 4350 1800
+NoConn ~ 4250 1800
+$Comp
+L Device:R_US R5
+U 1 1 5C09E9C9
+P 5300 950
+F 0 "R5" V 5400 900 50  0000 L CNN
+F 1 "100" V 5350 1050 50  0000 L CNN
+F 2 "Resistor_SMD:R_0805_2012Metric_Pad1.15x1.40mm_HandSolder" V 5340 940 50  0001 C CNN
+F 3 "~" H 5300 950 50  0001 C CNN
+	1    5300 950
+	0    1    1    0
+$EndComp
+Wire Wire Line
+	4750 950  4750 1050
+Wire Wire Line
+	4750 1050 4700 1050
+$Comp
+L Device:C C5
+U 1 1 5C09FAEE
+P 5100 1200
+F 0 "C5" H 5215 1246 50  0000 L CNN
+F 1 "100n" H 5215 1155 50  0000 L CNN
+F 2 "Capacitor_SMD:C_0805_2012Metric_Pad1.15x1.40mm_HandSolder" H 5138 1050 50  0001 C CNN
+F 3 "~" H 5100 1200 50  0001 C CNN
+	1    5100 1200
+	1    0    0    -1
+$EndComp
+Wire Wire Line
+	3150 850  5450 850
+Wire Wire Line
+	5450 850  5450 950
+Connection ~ 5450 850
+Wire Wire Line
+	5450 850  5800 850
+Wire Wire Line
+	5150 950  5100 950
+Wire Wire Line
+	5100 950  5100 1050
+Connection ~ 5100 950
+Wire Wire Line
+	5100 950  4750 950
+Wire Wire Line
+	4700 1200 4700 1350
+Wire Wire Line
+	4700 1350 5100 1350
+Wire Wire Line
+	4800 2150 5100 2150
+Wire Wire Line
+	5100 2150 5100 1350
+Connection ~ 5100 1350
+Wire Wire Line
+	5800 950  5800 1350
+Wire Wire Line
+	5800 1350 5100 1350
+Text Label 5400 1350 0    50   ~ 0
+VBAT_GND
+Text Label 5600 850  0    50   ~ 0
+VBAT
+$Comp
+L power:GND #PWR013
+U 1 1 5C0A4579
+P 3550 2300
+F 0 "#PWR013" H 3550 2050 50  0001 C CNN
+F 1 "GND" H 3555 2127 50  0000 C CNN
+F 2 "" H 3550 2300 50  0001 C CNN
+F 3 "" H 3550 2300 50  0001 C CNN
+	1    3550 2300
+	1    0    0    -1
+$EndComp
+Wire Wire Line
+	3750 2150 3750 2250
+Wire Wire Line
+	3550 2250 3550 2300
+Wire Wire Line
+	3750 2250 3550 2250
+Connection ~ 3750 2250
+Wire Wire Line
+	3950 1200 3700 1200
+$Comp
+L power:GND #PWR014
+U 1 1 5C0A805B
+P 3700 1500
+F 0 "#PWR014" H 3700 1250 50  0001 C CNN
+F 1 "GND" H 3705 1327 50  0000 C CNN
+F 2 "" H 3700 1500 50  0001 C CNN
+F 3 "" H 3700 1500 50  0001 C CNN
+	1    3700 1500
+	1    0    0    -1
+$EndComp
+NoConn ~ 3950 1050
+Wire Wire Line
+	4800 2250 4800 2150
+Connection ~ 4800 2150
 $EndSCHEMATC

Commit message: up
Parts:
- U5: footprint ESP32-footprints-Lib:ESP32-WROOM -> custom:esp32_wroom
Changed lines of the file:
@@
 F 0 "U5" H 6425 5937 60  0000 C CNN
 F 1 "ESP32-WROOM" H 6425 5831 60  0000 C CNN
-F 2 "ESP32-footprints-Lib:ESP32-WROOM" H 6800 5900 60  0001 C CNN
+F 2 "custom:esp32_wroom" H 6800 5900 60  0001 C CNN
 F 3 "" H 6000 5000 60  0001 C CNN
 	1    6450 4550

Commit message: Update schematic with vcc peripheral generation
Parts:
- added D4: LED_VCC33_PER, LEDs:LED_0805_HandSoldering, symbol Device:LED
- added R6, R8: 100k, Resistor_SMD:R_0805_2012Metric_Pad1.15x1.40mm_HandSolder, symbol Device:R_US
- added R7: 1k, Resistor_SMD:R_0805_2012Metric_Pad1.15x1.40mm_HandSolder, symbol Device:R_US
Connections:
- net +3V3: now also Q2.2 (S), R6.1
- net GND: now also D1.2 (A), D4.1 (K)
- net VREF_2.5: now reaches D1.1 (REF)
- net VREF_2.5: now also D1.3 (K), R7.2
- net VCC33_PER_CMD: now reaches Q2.1 (G)
- net VCC33_PER_CMD: now also R6.2
- net VCC33_PER: now reaches Q2.3 (D)
- net VCC33_PER: now also R7.1, R8.1
- new net: D4.2 (A), R8.2
Other:
- moved on the sheet: D1, Q2
Changed lines of the file:
@@
 L Reference_Voltage:TL431LP D1
 U 1 1 5BFCF494
-P 1350 4750
-F 0 "D1" V 1396 4681 50  0000 R CNN
-F 1 "TL431LP" V 1305 4681 50  0000 R CNN
-F 2 "Package_TO_SOT_THT:TO-92_Inline" H 1350 4600 50  0001 C CIN
-F 3 "http://www.ti.com/lit/ds/symlink/tl431.pdf" H 1350 4750 50  0001 C CIN
-	1    1350 4750
+P 1375 5850
+F 0 "D1" V 1421 5781 50  0000 R CNN
+F 1 "TL431LP" V 1330 5781 50  0000 R CNN
+F 2 "Package_TO_SOT_THT:TO-92_Inline" H 1375 5700 50  0001 C CIN
+F 3 "http://www.ti.com/lit/ds/symlink/tl431.pdf" H 1375 5850 50  0001 C CIN
+	1    1375 5850
 	0    -1   -1   0
 $EndComp
@@
 L Device:Q_NMOS_GSD Q2
 U 1 1 5BFD05AA
-P 3900 3100
-F 0 "Q2" H 4105 3146 50  0000 L CNN
-F 1 "SI2301" H 4105 3055 50  0000 L CNN
-F 2 "Package_TO_SOT_SMD:SOT-23" H 4100 3200 50  0001 C CNN
-F 3 "~" H 3900 3100 50  0001 C CNN
-	1    3900 3100
-	1    0    0    -1
+P 1750 4825
+F 0 "Q2" H 1955 4871 50  0000 L CNN
+F 1 "SI2301" H 1955 4780 50  0000 L CNN
+F 2 "Package_TO_SOT_SMD:SOT-23" H 1950 4925 50  0001 C CNN
+F 3 "~" H 1750 4825 50  0001 C CNN
+	1    1750 4825
+	0    1    -1   0
 $EndComp
 $Comp
@@
 	4800 2250 4800 2150
 Connection ~ 4800 2150
+Text Label 2600 2400 0    50   ~ 0
+VCC33
+Wire Wire Line
+	1200 4725 1375 4725
+$Comp
+L Device:R_US R6
+U 1 1 5C0EBD78
+P 1375 4875
+F 0 "R6" H 1443 4921 50  0000 L CNN
+F 1 "100k" H 1443 4830 50  0000 L CNN
+F 2 "Resistor_SMD:R_0805_2012Metric_Pad1.15x1.40mm_HandSolder" V 1415 4865 50  0001 C CNN
+F 3 "~" H 1375 4875 50  0001 C CNN
+	1    1375 4875
+	1    0    0    -1
+$EndComp
+Connection ~ 1375 4725
+Wire Wire Line
+	1375 4725 1550 4725
+Wire Wire Line
+	1750 5025 1375 5025
+Wire Wire Line
+	1375 5025 1200 5025
+Connection ~ 1375 5025
+Text Label 1200 4725 2    50   ~ 0
+VCC33
+Text Label 2300 4725 0    50   ~ 0
+VCC33_PER
+Text Label 1200 5025 2    50   ~ 0
+VCC33_PER_CMD
+Wire Wire Line
+	1950 4725 2125 4725
+$Comp
+L Device:R_US R7
+U 1 1 5C0F423B
+P 1375 5575
+F 0 "R7" H 1443 5621 50  0000 L CNN
+F 1 "1k" H 1443 5530 50  0000 L CNN
+F 2 "Resistor_SMD:R_0805_2012Metric_Pad1.15x1.40mm_HandSolder" V 1415 5565 50  0001 C CNN
+F 3 "~" H 1375 5575 50  0001 C CNN
+	1    1375 5575
+	1    0    0    -1
+$EndComp
+Wire Wire Line
+	1375 5425 1200 5425
+Text Label 1200 5425 2    50   ~ 0
+VCC33_PER
+$Comp
+L power:GND #PWR021
+U 1 1 5C0F80F9
+P 1375 6100
+F 0 "#PWR021" H 1375 5850 50  0001 C CNN
+F 1 "GND" H 1380 5927 50  0000 C CNN
+F 2 "" H 1375 6100 50  0001 C CNN
+F 3 "" H 1375 6100 50  0001 C CNN
+	1    1375 6100
+	1    0    0    -1
+$EndComp
+Wire Wire Line
+	1375 5925 1375 5950
+Connection ~ 1375 5950
+Wire Wire Line
+	1375 5950 1375 6100
+Wire Wire Line
+	1375 5725 1375 5750
+Wire Wire Line
+	1375 5750 1275 5750
+Wire Wire Line
+	1275 5750 1275 5850
+Connection ~ 1375 5750
+Wire Wire Line
+	1375 5750 1700 5750
+Text Label 1700 5750 0    50   ~ 0
+VREF_2.5
+$Comp
+L Device:R_US R8
+U 1 1 5C100C10
+P 2125 4875
+F 0 "R8" H 2193 4921 50  0000 L CNN
+F 1 "100k" H 2193 4830 50  0000 L CNN
+F 2 "Resistor_SMD:R_0805_2012Metric_Pad1.15x1.40mm_HandSolder" V 2165 4865 50  0001 C CNN
+F 3 "~" H 2125 4875 50  0001 C CNN
+	1    2125 4875
+	1    0    0    -1
+$EndComp
+Connection ~ 2125 4725
+Wire Wire Line
+	2125 4725 2300 4725
+$Comp
+L Device:LED D4
+U 1 1 5C100C98
+P 2125 5225
+F 0 "D4" V 2163 5107 50  0000 R CNN
+F 1 "LED_VCC33_PER" V 2072 5107 50  0000 R CNN
+F 2 "LEDs:LED_0805_HandSoldering" H 2125 5225 50  0001 C CNN
+F 3 "~" H 2125 5225 50  0001 C CNN
+	1    2125 5225
+	0    -1   -1   0
+$EndComp
+$Comp
+L power:GND #PWR022
+U 1 1 5C100DBB
+P 2125 5400
+F 0 "#PWR022" H 2125 5150 50  0001 C CNN
+F 1 "GND" H 2130 5227 50  0000 C CNN
+F 2 "" H 2125 5400 50  0001 C CNN
+F 3 "" H 2125 5400 50  0001 C CNN
+	1    2125 5400
+	1    0    0    -1
+$EndComp
+Wire Wire Line
+	2125 5025 2125 5075
+Wire Wire Line
+	2125 5375 2125 5400
 $EndSCHEMATC

Commit message: Changed LED
Parts:
- D1: footprint Package_TO_SOT_THT:TO-92_Inline -> Package_TO_SOT_SMD:SOT-23
- D4: footprint LEDs:LED_0805_HandSoldering -> LED_SMD:LED_0805_2012Metric
Changed lines of the file:
@@
 F 0 "D1" V 1421 5781 50  0000 R CNN
 F 1 "TL431LP" V 1330 5781 50  0000 R CNN
-F 2 "Package_TO_SOT_THT:TO-92_Inline" H 1375 5700 50  0001 C CIN
+F 2 "Package_TO_SOT_SMD:SOT-23" H 1375 5700 50  0001 C CIN
 F 3 "http://www.ti.com/lit/ds/symlink/tl431.pdf" H 1375 5850 50  0001 C CIN
 	1    1375 5850
@@
 F 0 "D4" V 2163 5107 50  0000 R CNN
 F 1 "LED_VCC33_PER" V 2072 5107 50  0000 R CNN
-F 2 "LEDs:LED_0805_HandSoldering" H 2125 5225 50  0001 C CNN
+F 2 "LED_SMD:LED_0805_2012Metric" H 2125 5225 50  0001 C CNN
 F 3 "~" H 2125 5225 50  0001 C CNN
 	1    2125 5225

Commit message: Adding sensoes
Parts:
- added R10, R9: 100k, Resistor_SMD:R_0805_2012Metric_Pad1.15x1.40mm_HandSolder, symbol Device:R_US
- added U6: HMC5883L, symbol custom_lib:HMC5883L
- added U7: BMP180, custom:BMP180, symbol custom_lib:BMP180
- added U8: DHT22, symbol custom_lib:DHT22
Connections:
- net GND: now also U6.2 (GND), U7.2 (GND), U8.4 (GND)
- net VCC33_PER: now also R10.1, R9.1, U6.1 (VCC), U7.1 (VCC), U8.1 (VCC)
- new net DHT: U8.2 (DATA)
- new net SCL: R10.2, U6.3 (SCL), U7.3 (SCL)
- new net SDA: R9.2, U6.4 (SDA), U7.4 (SDA)
- no-connect marks 5 -> 7
Changed lines of the file:
@@
 P 2600 2550
 F 0 "C3" H 2715 2596 50  0000 L CNN
-F 1 "10u" H 2715 2505 50  0000 L CNN
+F 1 "10u" H 2450 2450 50  0000 L CNN
 F 2 "Capacitor_SMD:CP_Elec_3x5.4" H 2638 2400 50  0001 C CNN
 F 3 "~" H 2600 2550 50  0001 C CNN
@@
 Text Label 1200 5025 2    50   ~ 0
 VCC33_PER_CMD
-Wire Wire Line
-	1950 4725 2125 4725
 $Comp
 L Device:R_US R7
@@
 	1    0    0    -1
 $EndComp
-Connection ~ 2125 4725
-Wire Wire Line
-	2125 4725 2300 4725
 $Comp
 L Device:LED D4
@@
 Wire Wire Line
 	2125 5375 2125 5400
+$Comp
+L custom_lib:HMC5883L U6
+U 1 1 5C119A33
+P 3200 3650
+F 0 "U6" H 3978 3222 60  0000 L CNN
+F 1 "HMC5883L" H 3978 3116 60  0000 L CNN
+F 2 "" H 3500 3550 60  0000 C CNN
+F 3 "" H 3500 3550 60  0000 C CNN
+	1    3200 3650
+	1    0    0    -1
+$EndComp
+$Comp
+L custom_lib:BMP180 U7
+U 1 1 5C119ACF
+P 3200 5750
+F 0 "U7" H 3778 6275 60  0000 L CNN
+F 1 "BMP180" H 3778 6169 60  0000 L CNN
+F 2 "custom:BMP180" H 3778 6063 60  0000 L CNN
+F 3 "" H 3200 5750 60  0000 C CNN
+	1    3200 5750
+	1    0    0    -1
+$EndComp
+$Comp
+L custom_lib:DHT22 U8
+U 1 1 5C119B9F
+P 3250 6800
+F 0 "U8" H 3728 7222 60  0000 L CNN
+F 1 "DHT22" H 3728 7116 60  0000 L CNN
+F 2 "" H 3250 6800 60  0000 C CNN
+F 3 "" H 3250 6800 60  0000 C CNN
+	1    3250 6800
+	1    0    0    -1
+$EndComp
+Wire Wire Line
+	3250 4600 2950 4600
+Wire Wire Line
+	3300 5750 2950 5750
+Wire Wire Line
+	3350 6800 3350 6850
+Wire Wire Line
+	3350 6850 2950 6850
+Text Label 2950 4600 2    50   ~ 0
+VCC33_PER
+Text Label 2950 5750 2    50   ~ 0
+VCC33_PER
+Text Label 2950 6850 2    50   ~ 0
+VCC33_PER
+$Comp
+L power:GND #PWR0101
+U 1 1 5C1233F4
+P 3400 5750
+F 0 "#PWR0101" H 3400 5500 50  0001 C CNN
+F 1 "GND" H 3405 5577 50  0000 C CNN
+F 2 "" H 3400 5750 50  0001 C CNN
+F 3 "" H 3400 5750 50  0001 C CNN
+	1    3400 5750
+	1    0    0    -1
+$EndComp
+$Comp
+L power:GND #PWR0102
+U 1 1 5C12369F
+P 3400 4600
+F 0 "#PWR0102" H 3400 4350 50  0001 C CNN
+F 1 "GND" H 3405 4427 50  0000 C CNN
+F 2 "" H 3400 4600 50  0001 C CNN
+F 3 "" H 3400 4600 50  0001 C CNN
+	1    3400 4600
+	1    0    0    -1
+$EndComp
+$Comp
+L power:GND #PWR0103
+U 1 1 5C1236EA
+P 3650 6800
+F 0 "#PWR0103" H 3650 6550 50  0001 C CNN
+F 1 "GND" H 3655 6627 50  0000 C CNN
+F 2 "" H 3650 6800 50  0001 C CNN
+F 3 "" H 3650 6800 50  0001 C CNN
+	1    3650 6800
+	1    0    0    -1
+$EndComp
+NoConn ~ 3550 6800
+Wire Wire Line
+	3550 4600 3550 4750
+Wire Wire Line
+	3550 4750 4050 4750
+Wire Wire Line
+	3700 4600 3700 4650
+Wire Wire Line
+	3700 4650 4050 4650
+Wire Wire Line
+	3500 5750 3500 5850
+Wire Wire Line
+	3500 5850 4050 5850
+Wire Wire Line
+	3600 5750 4050 5750
+Text Label 4050 4650 0    50   ~ 0
+SDA
+Text Label 4050 5750 0    50   ~ 0
+SDA
+Text Label 4050 4750 0    50   ~ 0
+SCL
+Text Label 4050 5850 0    50   ~ 0
+SCL
+Wire Wire Line
+	3450 6800 3450 7050
+Wire Wire Line
+	3450 7050 4000 7050
+Text Label 4000 7050 0    50   ~ 0
+DHT
+Text Label 2250 6150 2    50   ~ 0
+VCC33_PER
+Wire Wire Line
+	2250 6150 2300 6150
+Connection ~ 2125 4725
+Wire Wire Line
+	2125 4725 2300 4725
+Wire Wire Line
+	1950 4725 2125 4725
+$Comp
+L Device:R_US R9
+U 1 1 5C137FD7
+P 2300 6400
+F 0 "R9" H 2368 6446 50  0000 L CNN
+F 1 "100k" H 2368 6355 50  0000 L CNN
+F 2 "Resistor_SMD:R_0805_2012Metric_Pad1.15x1.40mm_HandSolder" V 2340 6390 50  0001 C CNN
+F 3 "~" H 2300 6400 50  0001 C CNN
+	1    2300 6400
+	1    0    0    -1
+$EndComp
+$Comp
+L Device:R_US R10
+U 1 1 5C138039
+P 2650 6400
+F 0 "R10" H 2718 6446 50  0000 L CNN
+F 1 "100k" H 2718 6355 50  0000 L CNN
+F 2 "Resistor_SMD:R_0805_2012Metric_Pad1.15x1.40mm_HandSolder" V 2690 6390 50  0001 C CNN
+F 3 "~" H 2650 6400 50  0001 C CNN
+	1    2650 6400
+	1    0    0    -1
+$EndComp
+Wire Wire Line
+	2300 6150 2300 6250
+Connection ~ 2300 6150
+Wire Wire Line
+	2300 6150 2650 6150
+Wire Wire Line
+	2650 6150 2650 6250
+Connection ~ 2650 6150
+Wire Wire Line
+	2650 6150 2750 6150
+Wire Wire Line
+	2300 6550 2050 6550
+Wire Wire Line
+	2650 6550 2650 6700
+Wire Wire Line
+	2650 6700 2050 6700
+Text Label 2050 6550 2    50   ~ 0
+SDA
+Text Label 2050 6700 2    50   ~ 0
+SCL
+NoConn ~ 3850 4600
 $EndSCHEMATC
